File: Eclise.kicad_pcb (KiCad board)
At the start: 2 copper layers, 19 parts, among them J1 Power Supply, J10 Sensor_Power, J11 Sensor_GND, J12 Sensor_Power, J13 Sensor_GND, J14 D12-D13, J2 AMS_In, J3 AMS_Out, J4 Prog_Pins, J5 Prog_Power, J6 A0-A3, J7 A4-A7, J8 D2-D5, J9 D6-D9, U1 ESP-01S

Commit message: ayaw kona
Parts:
- moved C1 117.8 mm to (161.1, 129.4), turned to 180 degrees
- moved J2 55.2 mm to (147.2, 139.0), turned to 180 degrees
- moved J6 50.6 mm to (156.8, 104.8), turned to 90 degrees
- moved U1 37.2 mm to (128.9, 120.5), turned to -90 degrees
- moved J1 27.4 mm to (157.5, 137.5)
- moved J3 19.5 mm to (127.2, 139.0), turned to 180 degrees
- moved J13 10.5 mm to (156.8, 66.3)
- moved J12 10.5 mm to (156.8, 83.0)
- moved R2 9.43 mm to (134.7, 106.8), turned to -90 degrees
- moved J14 7.61 mm to (156.8, 116.8)
- moved J5 7.33 mm to (140.6, 57.5)
- moved J4 7.23 mm to (122.0, 57.5)
- moved R1 0.64 mm to (132.1, 106.8), turned to -90 degrees
Routing:
- net GND: track 33.6 -> 406.4 mm
- net 5V: track 94.1 -> 225.6 mm
- net Net-(A1-D12_MISO): track 0.00 -> 34.7 mm
- net Net-(A1-D13_SCK): track 0.00 -> 33.7 mm
- net Net-(J6-Pin_4): track 59.5 -> 30.3 mm
- net Net-(J6-Pin_3): track 56.5 -> 29.8 mm
- net +3.3V: track 0.00 -> 20.8 mm
- net Net-(J6-Pin_2): track 50.5 -> 30.8 mm
- net E_RXD: track 2.53 -> 21.3 mm
- net Net-(J6-Pin_1): track 47.6 -> 31.8 mm
- net E_TXD: track 0.00 -> 11.5 mm
- net /TXO: track 29.9 -> 32.9 mm
- net Net-(J9-Pin_4): track 15.5 -> 18.0 mm
- net Net-(A1-D2_INT0): track 27.7 -> 25.5 mm
- net /RXI: track 40.0 -> 41.6 mm
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- added copper zone on B.Cu, net +3.3V
- added copper zone on B.Cu, net 5V
Other:
- board outline added: 80.2 x 96.8 mm

Commit message: final pcb
Parts:
- moved J3 7.81 mm to (124.3, 146.2)
- moved J2 7.81 mm to (144.3, 146.2)
Routing:
- net +3.3V: track 20.8 -> 32.0 mm
- net GND: track 406.4 -> 415.4 mm
- net 5V: track 225.6 -> 230.0 mm
Other:
- board size 80.2 x 96.8 mm -> 80.2 x 104.6 mm
Changed lines of the file:
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@@
 	(footprint "Connector_PinSocket_2.54mm:PinSocket_1x02_P2.54mm_Vertical"
 		(layer "F.Cu")
-		(at 147.2 139 180)
+		(at 144.275 146.24 180)
 		(descr "Through hole straight socket strip, 1x02, 2.54mm pitch, single row (from Kicad 4.0.7), script generated")
 		(tags "Through hole socket strip THT 1x02 2.54mm single row")
@@
 	(footprint "Connector_PinSocket_2.54mm:PinSocket_1x02_P2.54mm_Vertical"
 		(layer "F.Cu")
-		(at 127.2 139 180)
+		(at 124.275 146.24 180)
 		(descr "Through hole straight socket strip, 1x02, 2.54mm pitch, single row (from Kicad 4.0.7), script generated")
 		(tags "Through hole socket strip THT 1x02 2.54mm single row")
@@
 	(gr_rect
 		(start 88.25 49.25)
-		(end 168.5 146)
+		(end 168.5 153.85)
 		(stroke
 			(width 0.05)
@@
 	)
 	(segment
-		(start 127.2 136.46)
-		(end 147.2 136.46)
-		(width 1)
-		(layer "B.Cu")
-		(net "GND")
-	)
-	(segment
 		(start 134.7 107.825)
 		(end 134.7 106.76)
@@
 	)
 	(segment
+		(start 124.275 143.7)
+		(end 134.925 143.7)
+		(width 1)
+		(layer "B.Cu")
+		(net "GND")
+	)
+	(segment
 		(start 100.5 117.75)
 		(end 96.7 121.55)
@@
 	)
 	(segment
-		(start 140 136.46)
-		(end 147.2 136.46)
+		(start 157.5 137.5)
+		(end 150.75 137.5)
 		(width 1)
 		(layer "B.Cu")
@@
 	)
 	(segment
-		(start 90.775 140.9)
-		(end 93.35 143.475)
+		(start 100.275 150.4)
+		(end 90.775 140.9)
 		(width 1)
 		(layer "B.Cu")
@@
 	)
 	(segment
-		(start 156.7825 66.3)
-		(end 159.3 66.3)
+		(start 149.1 113.85)
+		(end 140.725 113.85)
 		(width 1)
 		(layer "B.Cu")
@@
 	)
 	(segment
-		(start 159.3 66.3)
-		(end 165.5 72.5)
-		(width 1)
+		(start 134.925 143.7)
+		(end 134.925 147.025)
+		(width 1.5)
 		(layer "B.Cu")
 		(net "GND")
 	)
 	(segment
-		(start 149.1 113.85)
-		(end 140.725 113.85)
+		(start 156.7825 66.3)
+		(end 159.3 66.3)
 		(width 1)
 		(layer "B.Cu")
@@
 	)
 	(segment
-		(start 163.29 143.46)
-		(end 147 143.46)
-		(width 1)
-		(layer "B.Cu")
-		(net "GND")
-	)
-	(segment
 		(start 113.545 89.045)
 		(end 114.95 90.45)
@@
 	)
 	(segment
-		(start 139.915 136.46)
-		(end 140 136.46)
-		(width 1)
-		(layer "B.Cu")
-		(net "GND")
-	)
-	(segment
-		(start 156.46 136.46)
-		(end 147.2 136.46)
+		(start 159.3 66.3)
+		(end 165.5 72.5)
 		(width 1)
 		(layer "B.Cu")
@@
 	)
 	(segment
-		(start 96.7 126.55)
-		(end 90.775 132.475)
+		(start 158.975 150.4)
+		(end 131.55 150.4)
 		(width 1)
 		(layer "B.Cu")
@@
 	)
 	(segment
-		(start 90.775 132.475)
-		(end 90.775 140.9)
+		(start 134.925 143.7)
+		(end 136.4 143.7)
 		(width 1)
 		(layer "B.Cu")
@@
 	)
 	(segment
+		(start 90.775 140.9)
+		(end 90.775 132.475)
+		(width 1)
+		(layer "B.Cu")
+		(net "GND")
+	)
+	(segment
 		(start 129.675 110.725)
 		(end 131 109.4)
@@
 	)
 	(segment
-		(start 165.5 72.5)
-		(end 165.5 141.25)
+		(start 136.4 143.7)
+		(end 144.275 143.7)
+		(width 1)
+		(layer "B.Cu")
+		(net "GND")
+	)
+	(segment
+		(start 134.925 147.025)
+		(end 131.55 150.4)
+		(width 1.5)
+		(layer "B.Cu")
+		(net "GND")
+	)
+	(segment
+		(start 90.775 132.475)
+		(end 96.7 126.55)
+		(width 1)
+		(layer "B.Cu")
+		(net "GND")
+	)
+	(segment
+		(start 150.75 137.5)
+		(end 144.55 143.7)
 		(width 1)
 		(layer "B.Cu")
@@
 	)
 	(segment
-		(start 93.35 143.475)
-		(end 132.9 143.475)
+		(start 144.55 143.7)
+		(end 144.275 143.7)
 		(width 1)
 		(layer "B.Cu")
@@
 	)
 	(segment
-		(start 132.9 143.475)
-		(end 139.915 136.46)
+		(start 165.5 72.5)
+		(end 165.5 143.875)
 		(width 1)
 		(layer "B.Cu")
@@
 	)
 	(segment
-		(start 151.2 115.95)
-		(end 149.1 113.85)
+		(start 165.5 143.875)
+		(end 158.975 150.4)
 		(width 1)
 		(layer "B.Cu")
@@
 	)
 	(segment
-		(start 165.5 141.25)
-		(end 163.29 143.46)
+		(start 151.2 115.95)
+		(end 149.1 113.85)
 		(width 1)
 		(layer "B.Cu")
@@
 	)
 	(segment
-		(start 147 143.46)
-		(end 140 136.46)
+		(start 131.55 150.4)
+		(end 100.275 150.4)
 		(width 1)
 		(layer "B.Cu")
@@
 	)
 	(segment
-		(start 153.65 140.9)
-		(end 151.75 139)
-		(width 1)
-		(layer "B.Cu")
-		(net "5V")
-	)
-	(segment
 		(start 139.075 52.325)
 		(end 128.9 52.325)
@@
 	)
 	(segment
-		(start 161.15 140.9)
-		(end 153.65 140.9)
-		(width 1)
-		(layer "B.Cu")
-		(net "5V")
-	)
-	(segment
 		(start 160.75 129.094887)
 		(end 160.75 81.8675)
@@
 	)
 	(segment
-		(start 162.5 139.55)
-		(end 161.15 140.9)
+		(start 161.055113 129.4)
+		(end 160.75 129.094887)
 		(width 1)
 		(layer "B.Cu")
@@
 	)
 	(segment
-		(start 162.5 137.5)
-		(end 162.5 139.55)
+		(start 156.8325 72.95)
+		(end 156.8325 82.95)
 		(width 1)
 		(layer "B.Cu")
@@
 	)
 	(segment
-		(start 161.055113 129.4)
-		(end 160.75 129.094887)
+		(start 155.81 146.24)
+		(end 144.275 146.24)
 		(width 1)
 		(layer "B.Cu")
@@
 	)
 	(segment
-		(start 156.8325 72.95)
-		(end 156.8325 82.95)
+		(start 99.3 52.325)
+		(end 128.9 52.325)
 		(width 1)
 		(layer "B.Cu")
@@
 	)
 	(segment
-		(start 99.3 52.325)
-		(end 128.9 52.325)
+		(start 150.75 82.95)
+		(end 144.655 89.045)
 		(width 1)
 		(layer "B.Cu")
@@
 	)
 	(segment
-		(start 150.75 82.95)
-		(end 144.655 89.045)
+		(start 162.5 139.55)
+		(end 155.81 146.24)
 		(width 1)
 		(layer "B.Cu")
@@
 	)
 	(segment
-		(start 151.75 139)
-		(end 147.2 139)
+		(start 162.5 137.5)
+		(end 162.5 139.55)
 		(width 1)
 		(layer "B.Cu")
@@
 	)
 	(segment
-		(start 125 139)
-		(end 122.5 136.5)
+		(start 120.39 146.24)
+		(end 124.275 146.24)
 		(width 1)
 		(layer "B.Cu")
@@
 	)
 	(segment
-		(start 127.2 139)
-		(end 125 139)
+		(start 117.475 136.995)
+		(end 117.475 143.325)
 		(width 1)
 		(layer "B.Cu")
@@
 	)
 	(segment
-		(start 122.5 132)
-		(end 126.35 128.15)
+		(start 117.475 143.325)
+		(end 120.39 146.24)
 		(width 1)
 		(layer "B.Cu")
@@
 	)
 	(segment
-		(start 122.5 136.5)
-		(end 122.5 132)
+		(start 126.35 128.12)
+		(end 117.475 136.995)
 		(width 1)
 		(layer "B.Cu")

Commit message: Rearrangement of PCB
Parts:
- moved J12 28.6 mm to (179.1, 65.0)
- moved J13 27.4 mm to (179.0, 82.4)
- moved J14 22.2 mm to (179.0, 117.0)
- moved J6 22.2 mm to (179.0, 104.8)
- moved C1 21.0 mm to (181.3, 135.1)
- moved J1 21.0 mm to (177.8, 143.2)
- moved A1 19.9 mm to (138.4, 87.3)
- moved R1 19.4 mm to (150.8, 101.5)
- moved R2 19.4 mm to (153.3, 101.4)
- moved U1 16.6 mm to (145.5, 119.5)
- moved J5 14.3 mm to (154.8, 59.2)
- moved J2 9.56 mm to (153.0, 142.3)
- moved J3 9.56 mm to (133.0, 142.3)
- moved J4 7.70 mm to (129.5, 59.3)
- moved J7 4.31 mm to (96.8, 141.5)
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Connections:
- A1 pad GND4: (no net) -> GND
- J4 pad 2: /TXO -> /RXI
- J4 pad 3: /RXI -> /TXO
Routing:
- net 5V: track 230.0 -> 303.4 mm
- net Net-(A1-A5/SCL): track 57.5 -> 99.5 mm
- net GND: track 415.4 -> 454.2 mm
- net /RXI: track 41.6 -> 20.2 mm
- net Net-(J9-Pin_4): track 18.0 -> 37.3 mm
- net Net-(J9-Pin_3): track 17.4 -> 36.3 mm
- net Net-(J7-Pin_4): track 33.9 -> 52.2 mm
- net Net-(J7-Pin_3): track 34.9 -> 53.1 mm
- net Net-(J9-Pin_2): track 18.0 -> 35.3 mm
- net /DTR: track 25.0 -> 41.3 mm
- net Net-(J9-Pin_1): track 18.2 -> 34.2 mm
- net Net-(J8-Pin_4): track 20.0 -> 34.4 mm
- net Net-(J8-Pin_3): track 22.5 -> 35.4 mm
- net Net-(A1-D3_INT1): track 24.0 -> 36.4 mm
- net Net-(A1-D2_INT0): track 25.5 -> 37.4 mm
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Other:
- board size 80.2 x 104.6 mm -> 101.6 x 101.6 mm

Commit message: Fixed AMS pins placment
Parts:
- moved J2 9.63 mm to (161.6, 138.0), turned to 0 degrees
- moved J3 9.63 mm to (141.6, 138.0), turned to 0 degrees
Routing:
- net 5V: track 303.4 -> 275.9 mm
- net +3.3V: track 33.6 -> 16.5 mm
- net GND: track 454.2 -> 445.6 mm

Commit message: revised pcb
Parts:
- removed J11, J13: Sensor_GND, TerminalBlock:TerminalBlock_MaiXu_MX126-5.0-03P_1x03_P5.00mm
- removed J12: Sensor_Power, TerminalBlock:TerminalBlock_MaiXu_MX126-5.0-03P_1x03_P5.00mm
- removed J14: D12-D13, TerminalBlock:TerminalBlock_MaiXu_MX126-5.0-02P_1x02_P5.00mm
- removed J4: Prog_Pins, TerminalBlock:TerminalBlock_MaiXu_MX126-5.0-03P_1x03_P5.00mm
- removed J5: Prog_Power, TerminalBlock:TerminalBlock_MaiXu_MX126-5.0-03P_1x03_P5.00mm
- J10: value Sensor_Power -> OLED; footprint TerminalBlock:TerminalBlock_MaiXu_MX126-5.0-03P_1x03_P5.00mm -> TerminalBlock:TerminalBlock_MaiXu_MX126-5.0-04P_1x04_P5.00mm
- J6: value A0-A3 -> DHT; footprint TerminalBlock:TerminalBlock_MaiXu_MX126-5.0-04P_1x04_P5.00mm -> TerminalBlock:TerminalBlock_MaiXu_MX126-5.0-03P_1x03_P5.00mm
- J7: value A4-A7 -> Ultrasonic
- J8: value D2-D5 -> MQ2
- J9: value D6-D9 -> Servo; footprint TerminalBlock:TerminalBlock_MaiXu_MX126-5.0-04P_1x04_P5.00mm -> TerminalBlock:TerminalBlock_MaiXu_MX126-5.0-03P_1x03_P5.00mm
- moved J1 129.8 mm to (87.2, 50.3), turned to -90 degrees
- moved C1 119.0 mm to (94.8, 53.5), turned to 90 degrees
- moved J6 84.3 mm to (103.2, 67.8), turned to 180 degrees
- moved J10 78.5 mm to (172.8, 75.0), turned to 90 degrees
- moved J8 63.7 mm to (107.6, 138.0), turned to 0 degrees
- moved J7 58.7 mm to (91.5, 83.0), turned to -90 degrees
- moved J9 20.4 mm to (91.5, 116.5)
- moved A1 7.92 mm to (130.8, 89.5)
- moved U1 6.21 mm to (150.7, 116.1)
- moved J2 4.96 mm to (166.5, 137.2)
- moved J3 4.96 mm to (146.5, 137.2)
- moved R2 4.85 mm to (158.2, 101.3)
- moved R1 1.66 mm to (152.4, 101.3)
Connections:
- A1 pad A0: Net-(J6-Pin_1) -> MQ2_A0
- A1 pad A4: Net-(A1-A4/SDA) -> OLED_SDA
- A1 pad A5: Net-(A1-A5/SCL) -> OLED_SCL
- A1 pad D4: Net-(J8-Pin_3) -> DHT_Data
- A1 pad D5: Net-(J8-Pin_4) -> MQ2_D5
- A1 pad D6: Net-(J9-Pin_1) -> Trig
- A1 pad D7: Net-(J9-Pin_2) -> Echo
- A1 pad D9: Net-(J9-Pin_4) -> Servo_PWM
- J10 pad 1: 5V -> GND
- J10 pad 3: 5V -> OLED_SCL
- J6 pad 1: Net-(J6-Pin_1) -> DHT_Data
- J6 pad 2: Net-(J6-Pin_2) -> 5V
- J6 pad 3: Net-(J6-Pin_3) -> GND
- J7 pad 1: Net-(A1-A4/SDA) -> 5V
- J7 pad 2: Net-(A1-A5/SCL) -> Trig
- J7 pad 3: Net-(J7-Pin_3) -> Echo
- J7 pad 4: Net-(J7-Pin_4) -> GND
- J8 pad 1: Net-(A1-D2_INT0) -> 5V
- J8 pad 2: Net-(A1-D3_INT1) -> GND
- J8 pad 3: Net-(J8-Pin_3) -> MQ2_D5
- J8 pad 4: Net-(J8-Pin_4) -> MQ2_A0
- J9 pad 1: Net-(J9-Pin_1) -> Servo_PWM
- J9 pad 2: Net-(J9-Pin_2) -> GND
- J9 pad 3: Net-(J9-Pin_3) -> 5V
Routing:
- net GND: track 445.6 -> 332.2 mm
- net Net-(A1-A5/SCL): track 99.5 -> 0.00 mm
- net Net-(A1-A4/SDA): track 77.9 -> 0.00 mm
- net OLED_SDA: track 0.00 -> 62.6 mm
- net Net-(J7-Pin_3): track 53.1 -> 0.00 mm
- net MQ2_A0: track 0.00 -> 52.9 mm
- net Net-(J7-Pin_4): track 52.2 -> 0.00 mm
- net MQ2_D5: track 0.00 -> 52.0 mm
- net 5V: track 275.9 -> 327.7 mm
- net OLED_SCL: track 0.00 -> 49.1 mm
- net /DTR: track 41.3 -> 0.00 mm
- net Net-(A1-D12_MISO): track 41.1 -> 0.00 mm
- net Net-(A1-D13_SCK): track 40.1 -> 0.00 mm
- net Net-(J6-Pin_1): track 38.1 -> 0.00 mm
- net Net-(A1-D2_INT0): track 37.4 -> 0.00 mm
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- removed copper zone on B.Cu, net +3.3V
- removed copper zone on B.Cu, net 5V
